File: tamagotchi.kicad_sch (KiCad schematic)
At the start: 7 parts, among them SW1 SW_Push, SW2 SW_Push, SW3 SW_Push, U1 XIAO-ESP32-C3-SMD, U2 HS96L03W2C03

Commit message: Add files via upload
Parts:
- removed U2: HS96L03W2C03, easyeda2kicad:OLED-TH_L27.8-W27.2-P2.54_C9900033791, symbol easyeda2kicad:HS96L03W2C03
- added LCD1: HS180S10B, easyeda2kicad:LCD-TH_L51.0-W35.0-P2.54_HS180S10B, symbol easyeda2kicad:HS180S10B
- U1: footprint New_XIAO_Series_Footprints:XIAO-ESP32-C3-SMD -> New_XIAO_Series_Footprints:XIAO-ESP32-C3-DIP-SMD
Connections:
- net +3V3: now also LCD1.11 (VCC), LCD1.13 (BLA)
- net GND: now also LCD1.12 (GND)
- net at BUZZER1.1 (+): now also U1.4 (GPIO5_A3_D3); no longer U1.11 (GPIO10_D10_MOSI)
- net DC: now reaches U1.6 (GPIO7_D5_SCL)
- net DC: now also LCD1.18 (DC)
- net RES: now reaches U1.5 (GPIO6_D4_SDA)
- net RES: now also LCD1.19 (RES)
- net CS1: now reaches U1.7 (GPIO21_D6_TX)
- net CS1: now also LCD1.20 (CS1)
- net at U1.9 (GPIO8_D8_SCK): now also LCD1.16 (CLK)
- new net: LCD1.17 (SDA), U1.11 (GPIO10_D10_MOSI)
- no-connect marks 11 -> 20
Other:
- moved on the sheet: BUZZER1, SW1, SW2, SW3
